File: qa/data/kichad/kds_live_apply/live_apply.kicad_pcb (KiCad board)
At the start: 2 copper layers, 0 parts

Commit message: Place schematic footprints from KDS safely
Parts:
- added R1: 1k, Resistor_SMD:R_0603_1608Metric, F.Cu at (10.0, 10.0)
Changed lines of the file:
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@@
   (net 0 "")
   (net 1 "Net1")
+  (footprint "Resistor_SMD:R_0603_1608Metric"
+    (layer "F.Cu")
+    (at 10 10)
+    (property "Reference" "R1"
+      (at 0 -1.5 0)
+      (layer "F.SilkS")
+      (effects (font (size 1 1) (thickness 0.15)))
+    )
+    (property "Value" "1k"
+      (at 0 1.5 0)
+      (layer "F.Fab")
+      (effects (font (size 1 1) (thickness 0.15)))
+    )
+    (property "Datasheet" ""
+      (at 0 0 0)
+      (layer "F.Fab")
+      (hide yes)
+      (effects (font (size 1 1) (thickness 0.15)))
+    )
+    (property "Description" "Live KDS placement fixture"
+      (at 0 0 0)
+      (layer "F.Fab")
+      (hide yes)
+      (effects (font (size 1 1) (thickness 0.15)))
+    )
+    (sheetname "/")
+    (sheetfile "live_apply.kicad_sch")
+    (attr smd)
+    (fp_line
+      (start -0.5 -0.5)
+      (end 0.5 -0.5)
+      (stroke (width 0.12) (type solid))
+      (layer "F.SilkS")
+    )
+    (pad "1" smd roundrect
+      (at -0.8 0)
+      (size 0.9 0.95)
+      (layers "F.Cu" "F.Paste" "F.Mask")
+      (roundrect_rratio 0.25)
+      (net 1 "Net1")
+    )
+    (pad "2" smd roundrect
+      (at 0.8 0)
+      (size 0.9 0.95)
+      (layers "F.Cu" "F.Paste" "F.Mask")
+      (roundrect_rratio 0.25)
+    )
+  )
   (net_class "Default" ""
     (clearance 0.2)
