File: qa/data/kichad/kds_live_apply/live_apply.kicad_pcb (KiCad board)
At the start: 2 copper layers, 1 part

Commit message: Own generated KDS footprints deterministically
Other:
- net class Default removed
Changed lines of the file:
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@@
-(kicad_pcb (version 20240108) (generator "pcbnew")
-  (general
-    (thickness 1.6)
-  )
-  (paper "A4")
-  (layers
-    (0 "F.Cu" signal)
-    (31 "B.Cu" signal)
-    (37 "F.SilkS" user "F.Silkscreen")
-    (40 "Dwgs.User" user "User.Drawings")
-    (44 "Edge.Cuts" user)
-  )
-  (setup
-    (pad_to_mask_clearance 0)
-    (allow_soldermask_bridges_in_footprints no)
-  )
-  (net 0 "")
-  (net 1 "Net1")
-  (footprint "Resistor_SMD:R_0603_1608Metric"
-    (layer "F.Cu")
-    (at 10 10)
-    (property "Reference" "R1"
-      (at 0 -1.5 0)
-      (layer "F.SilkS")
-      (effects (font (size 1 1) (thickness 0.15)))
-    )
-    (property "Value" "1k"
-      (at 0 1.5 0)
-      (layer "F.Fab")
-      (effects (font (size 1 1) (thickness 0.15)))
-    )
-    (property "Datasheet" ""
-      (at 0 0 0)
-      (layer "F.Fab")
-      (hide yes)
-      (effects (font (size 1 1) (thickness 0.15)))
-    )
-    (property "Description" "Live KDS placement fixture"
-      (at 0 0 0)
-      (layer "F.Fab")
-      (hide yes)
-      (effects (font (size 1 1) (thickness 0.15)))
-    )
-    (sheetname "/")
-    (sheetfile "live_apply.kicad_sch")
-    (attr smd)
-    (fp_line
-      (start -0.5 -0.5)
-      (end 0.5 -0.5)
-      (stroke (width 0.12) (type solid))
-      (layer "F.SilkS")
-    )
-    (pad "1" smd roundrect
-      (at -0.8 0)
-      (size 0.9 0.95)
-      (layers "F.Cu" "F.Paste" "F.Mask")
-      (roundrect_rratio 0.25)
-      (net 1 "Net1")
-    )
-    (pad "2" smd roundrect
-      (at 0.8 0)
-      (size 0.9 0.95)
-      (layers "F.Cu" "F.Paste" "F.Mask")
-      (roundrect_rratio 0.25)
-    )
-  )
-  (net_class "Default" ""
-    (clearance 0.2)
-    (trace_width 0.25)
-    (via_dia 0.8)
-    (via_drill 0.4)
-    (uvia_dia 0.3)
-    (uvia_drill 0.1)
-  )
+(kicad_pcb
+	(version 20260206)
+	(generator "pcbnew")
+	(generator_version "10.0")
+	(general
+		(thickness 1.6)
+		(legacy_teardrops no)
+	)
+	(paper "A4")
+	(layers
+		(0 "F.Cu" signal)
+		(2 "B.Cu" signal)
+		(5 "F.SilkS" user "F.Silkscreen")
+		(17 "Dwgs.User" user "User.Drawings")
+		(25 "Edge.Cuts" user)
+		(27 "Margin" user)
+		(31 "F.CrtYd" user "F.Courtyard")
+		(29 "B.CrtYd" user "B.Courtyard")
+	)
+	(setup
+		(pad_to_mask_clearance 0)
+		(allow_soldermask_bridges_in_footprints no)
+		(tenting
+			(front yes)
+			(back yes)
+		)
+		(covering
+			(front no)
+			(back no)
+		)
+		(plugging
+			(front no)
+			(back no)
+		)
+		(capping no)
+		(filling no)
+		(pcbplotparams
+			(layerselection 0x00000000_00000000_55555555_5755f5ff)
+			(plot_on_all_layers_selection 0x00000000_00000000_00000000_00000000)
+			(disableapertmacros no)
+			(usegerberextensions no)
+			(usegerberattributes yes)
+			(usegerberadvancedattributes yes)
+			(creategerberjobfile yes)
+			(dashed_line_dash_ratio 12)
+			(dashed_line_gap_ratio 3)
+			(svgprecision 4)
+			(plotframeref no)
+			(mode 1)
+			(useauxorigin no)
+			(pdf_front_fp_property_popups yes)
+			(pdf_back_fp_property_popups yes)
+			(pdf_metadata yes)
+			(pdf_single_document no)
+			(dxfpolygonmode yes)
+			(dxfimperialunits yes)
+			(dxfusepcbnewfont yes)
+			(psnegative no)
+			(psa4output no)
+			(plot_black_and_white yes)
+			(sketchpadsonfab no)
+			(plotpadnumbers no)
+			(hidednponfab no)
+			(sketchdnponfab yes)
+			(crossoutdnponfab yes)
+			(subtractmaskfromsilk no)
+			(outputformat 1)
+			(mirror no)
+			(drillshape 1)
+			(scaleselection 1)
+			(outputdirectory "")
+		)
+	)
+	(footprint "Resistor_SMD:R_0603_1608Metric"
+		(layer "F.Cu")
+		(at 10 10)
+		(property "Reference" "R1"
+			(at 0 -1.5 0)
+			(layer "F.SilkS")
+			(effects
+				(font
+					(size 1 1)
+					(thickness 0.15)
+				)
+			)
+		)
+		(property "Value" "1k"
+			(at 0 1.5 0)
+			(layer "F.Fab")
+			(effects
+				(font
+					(size 1 1)
+					(thickness 0.15)
+				)
+			)
+		)
+		(property "Datasheet" ""
+			(at 0 0 0)
+			(layer "F.Fab")
+			(hide yes)
+			(effects
+				(font
+					(size 1 1)
+					(thickness 0.15)
+				)
+			)
+		)
+		(property "Description" "Live KDS placement fixture"
+			(at 0 0 0)
+			(layer "F.Fab")
+			(hide yes)
+			(effects
+				(font
+					(size 1 1)
+					(thickness 0.15)
+				)
+			)
+		)
+		(sheetname "/")
+		(sheetfile "live_apply.kicad_sch")
+		(attr smd)
+		(duplicate_pad_numbers_are_jumpers no)
+		(fp_line
+			(start -0.5 -0.5)
+			(end 0.5 -0.5)
+			(stroke
+				(width 0.12)
+				(type solid)
+			)
+			(layer "F.SilkS")
+		)
+		(pad "1" smd roundrect
+			(at -0.8 0)
+			(size 0.9 0.95)
+			(layers "F.Cu" "F.Mask" "F.Paste")
+			(roundrect_rratio 0.25)
+			(net "Net1")
+		)
+		(pad "2" smd roundrect
+			(at 0.8 0)
+			(size 0.9 0.95)
+			(layers "F.Cu" "F.Mask" "F.Paste")
+			(roundrect_rratio 0.25)
+		)
+		(embedded_fonts no)
+	)
+	(embedded_fonts no)
 )
